File: NXP_K22_TestBoard/microcontroller.kicad_sch (KiCad schematic)
At the start: 41 parts, among them SW201 SW_Push, U201 AMS1117-3.3, U202 MK22FN512, U203 W25Q32JVSS, X201 ECS-TXO-3225MV, Y201 Crystal

Commit message: Finished board layout
Design rules not checked yet
Parts:
- C201, C205: MPN (none) -> Generic C/1uF/X7R/50V/0603
- C202, C203: value C -> 20p; MPN (none) -> Generic C/12pF/C0G/50V/0603
- C204: LCSC Part # (none) -> C122325; MPN (none) -> T495D226K035ATE125
- C206, C207, C208, C209, C211, C212, C213, C214, C219: MPN (none) -> Generic C/100nF/X7R/16V/0603
- C210: MPN (none) -> Generic C/1nF/X7R/16V/0603
- C216: MPN (none) -> Generic C/10pF/C0G/50V/0603
- C217: value 1nF -> 1n; MPN (none) -> Generic C/1nF/X7R/16V/0603
- C218: value 100nF -> 100n; MPN (none) -> Generic C/100nF/X7R/16V/0603
- FB201: LCSC Part # (none) -> C275489; MPN (none) -> MPZ1608Y221BTA00
- R201, R202, R206: MPN (none) -> Generic R/33R/0603
- R203, R204, R205: MPN (none) -> Generic R/10k/0603
- SW201: LCSC Part # (none) -> C221869
- U201: LCSC Part # (none) -> C6186; MPN (none) -> AMS1117-3.3
- U202: Champ5 (none) -> C965554; MPN (none) -> MK22FN512VLH12
- U203: LCSC Part # (none) -> C179173; MPN (none) -> W25Q32JVSSIQ
- X201: LCSC Part # (none) -> C5355149; MPN (none) -> ECS-TXO-3225MV-122.8-TR
- Y201: value Crystal -> 32.768 kHz; LCSC Part # (none) -> C32346; MPN (none) -> Q13FC1350000400
